File: ActivePrecharge RevB/Analog.kicad_sch (KiCad schematic)
At the start: 32 parts, among them IC1 AMC1350DWVR, IC2 AMC1350DWVR, U2 TLV9001IDBVR, U3 TLV9001IDBVR

Commit message: With Ravi comments
Parts:
- removed C15: 10n, symbol Device:C
- removed R15: 10, symbol Device:R_US
- removed U2: TLV9001IDBVR, TLV9001IDBVR:SOT95P280X145-5N, symbol 2G5-OPAMP:TLV9001IDBVR
- added C17: 10nF, symbol Device:C
- added R13: 10, symbol Device:R_US
- added U4: TLV9001IDBVR, DBV0005A_N, symbol 2G5-OPAMP:TLV9001IDBVR
- C10, C11, C12, C3, C4, C9: P/N (none) -> MLASU168SB5105KTNA01
- C13, C14, C5, C6: P/N (none) -> MLASH168SB7104KTNA01
- C16: value 10n -> 10nF; P/N (none) -> MSASH168SB5103KTNA01
- C7, C8: P/N (none) -> MLASU063SB7102KFNA01
- R10, R8: value 2.5k -> 2.49k; P/N (none) -> CRCW0603100KFKEE
- R11: P/N (none) -> CRCW060315K0FKEA
- R12: P/N (none) -> CRCW060310K0FKEI
- R14: renamed from R13; P/N (none) -> CRCW060315K0FKEA
- R15: renamed from R14; P/N (none) -> CRCW060310K0FKEI
- R7, R9: value 105k -> 100k; P/N (none) -> CRCW0603100KFKEE
- U3: footprint TLV9001IDBVR:SOT95P280X145-5N -> DBV0005A_N
Connections:
- net 3V3: now also U4.5 (V+)
- net LVGND: now also C17.2, U4.2 (V-)
- net V1: now also U3.3 (IN+)
- net V2: now also U4.3 (IN+); no longer U3.1 (IN+)
- net VOut1: now also C16.1, R13.2
- net VOut2: now also C17.1; no longer C16.1
- net at R14.1, R16.1: now also U4.1 (OUT); no longer U3.4 (OUT)
- net at R14.2, R15.1: now also U4.4 (IN-); no longer U3.3 (IN-)
- net at R11.2, R12.1: now also U3.4 (IN-)
- net at R11.1: now also U3.1 (OUT), R13.1
- net REG_PWR renamed REG_3V3
Other:
- note added: "Isolating amplifiers with a fixed gain of 0.4"
- note added: "Op-amps with a gain of 2.5"
- note added: "Voltage dividers to convert 120V to 3.3V Note: Isolated amplifier takes up to 5V"
- moved on the sheet: C10, C11, C12, C13, C14, C3, C4, C5, C6, C7, C8, C9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
