File: Hardware/Analog.kicad_sch (KiCad schematic)
At the start: 42 parts, among them IC1 AMC1350DWVR, IC2 AMC1350DWVR, IC3 ZXRE160AET5TA, U2 TLV9001IDBVR, U3 TLV9001IDBVR

Commit message: submodules
Parts:
- renumbered C6 to C1, C21 to C10, C14 to C11, C15 to C12, C16 to C13, C17 to C14, C22 to C15, C23 to C16, C7 to C2, C20 to C3, C8 to C4, C9 to C5, C10 to C6, C11 to C7, C12 to C8, C13 to C9, IC3 to IC1, IC1 to IC2, IC2 to IC3, R8 to R1, R26 to R10, R27 to R11, R24 to R12, R28 to R13, R22 to R14, R29 to R15, R25 to R16, R30 to R17, R9 to R2, R10 to R3, R11 to R4, R18 to R5, R19 to R6, R20 to R7, R21 to R8, R23 to R9, TP6 to TP1, TP7 to TP2, TP8 to TP3, TP9 to TP4, U2 to U1, U3 to U2

Commit message: Fixed this shit finally im free
Parts:
- removed C10: 0.47uF, Capacitor_SMD:C_0603_1608Metric_Pad1.08x0.95mm_HandSolder, symbol Device:C_Small
- removed C12, C9: 1uF, Capacitor_SMD:C_0603_1608Metric_Pad1.08x0.95mm_HandSolder, symbol Device:C_Small
- removed C14, C3, C5: 100nF, Capacitor_SMD:C_0603_1608Metric_Pad1.08x0.95mm_HandSolder, symbol Device:C_Small
- removed C15, C16: 10nF, Capacitor_SMD:C_0603_1608Metric_Pad1.08x0.95mm_HandSolder, symbol Device:C
- removed C2: 1uF, Capacitor_SMD:C_0603_1608Metric_Pad1.08x0.95mm_HandSolder, symbol Device:C
- removed C7: 1nF, Capacitor_SMD:C_0603_1608Metric_Pad1.08x0.95mm_HandSolder, symbol Device:C_Small
- removed IC1: ZXRE160AET5TA, ActivePrecharge-RevB:SOT95P280X100-5N, symbol VREF:ZXRE160AET5TA
- removed IC3: AMC1350DWVR, ActivePrecharge-RevB:SOIC127P1150X280-8N, symbol AMC1350:AMC1350DWVR
- removed R10, R11, R4, R8, R9: 2.49k, Resistor_SMD:R_0603_1608Metric_Pad0.98x0.95mm_HandSolder, symbol Device:R_US
- removed R12, R13, R14, R15, R7: 15k, Resistor_SMD:R_0603_1608Metric_Pad0.98x0.95mm_HandSolder, symbol Device:R_US
- removed R16, R17: 10, Resistor_SMD:R_0603_1608Metric_Pad0.98x0.95mm_HandSolder, symbol Device:R_US
- removed R3: 100k, Resistor_SMD:R_0603_1608Metric_Pad0.98x0.95mm_HandSolder, symbol Device:R_US
- removed R5: 1k, Resistor_SMD:R_0603_1608Metric_Pad0.98x0.95mm_HandSolder, symbol Device:R_US
- removed R6: 5.1k, Resistor_SMD:R_0603_1608Metric_Pad0.98x0.95mm_HandSolder, symbol Device:R_US
- removed TP1: Vin1, TestPoint:TestPoint_THTPad_D1.0mm_Drill0.5mm, symbol Connector:TestPoint
- removed TP2: Vin2, TestPoint:TestPoint_THTPad_D1.0mm_Drill0.5mm, symbol Connector:TestPoint
- removed TP4: V2, TestPoint:TestPoint_THTPad_D1.0mm_Drill0.5mm, symbol Connector:TestPoint
- removed U1, U2: TLV9001IDBVR, ActivePrecharge-RevB:DBV0005A_N, symbol Simulation_SPICE:OPAMP
- added TP6: Vin, TestPoint:TestPoint_Keystone_5005-5009_Compact, symbol Connector:TestPoint
- added TP8: V-, TestPoint:TestPoint_Keystone_5005-5009_Compact, symbol Connector:TestPoint
- TP7: renamed from TP3; value V1 -> V+; footprint TestPoint:TestPoint_THTPad_D1.0mm_Drill0.5mm -> TestPoint:TestPoint_Keystone_5005-5009_Compact; now left out of the parts list
- renumbered C4 to C10, C6 to C11, C8 to C12, C11 to C13, C13 to C14, C1 to C9, IC2 to IC1, R1 to R20, R2 to R21
Connections:
- net LVGND: no longer IC1.6 (OUTN)
- net HV+ renamed HV
- net V1 renamed V+
- net Vin1 renamed Vin
- net Vin: now also TP6.1
- new net V-: IC1.6 (OUTN), TP8.1
Other:
- note removed: "Op-amps that subtract an offset of 0.8V and apply a gain of 6.425 to create a 0.34V to 3.36V output range"
- note removed: "Voltage reference chip that creates a stable 0.8V reference"
- moved on the sheet: C10, C11, C12, C13, C14, C9, IC1, R20, R21, TP7

Commit message: added some silkscreen stuff and gerbers + bom etc
Parts:
- TP6: now left out of the parts list
Changed lines of the file:
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@@
 		(unit 1)
 		(exclude_from_sim no)
-		(in_bom yes)
+		(in_bom no)
 		(on_board yes)
 		(dnp no)
