File: Hardware/ActivePrecharge RevB.kicad_pcb (KiCad board)
At the start: 2 copper layers, 96 x 57 mm, 91 parts, among them IC1 AMC1350DWVR, IC2 AMC1350DWVR, J1 HVConnector, J2 PrechargeContactor, J3 MainContactor, J4 ExportConnector, J5 HV+, J6 HV-, J7 Conn_01x02_Pin, U1 TLV9002QDRQ1, U2 LT1963AEST-3.3#TRPBF

Commit message: changed fuses to be HV fuses
Parts:
- removed the G*** at (341.0, 70.8)
- removed J7: Conn_01x02_Pin, Connector_PinHeader_2.54mm:PinHeader_1x02_P2.54mm_Vertical
- added G***: LOGO, LOGO, B.Cu at (121.2, 96.5)
- added TP12: 3v3, TestPoint:TestPoint_Keystone_5005-5009_Compact, F.Cu at (174.5, 82.8)
- added TP13: GND, TestPoint:TestPoint_Keystone_5005-5009_Compact, F.Cu at (189.8, 124.8)
- F1, F2: footprint ActivePrecharge-RevB:FUSE_3568 -> UTSVT-Power:HV-Fuse
- LOGO1: moved to B.Cu
- moved LOGO1 65.2 mm to (181.2, 87.6), turned to 180 degrees
- moved D1 12.6 mm to (121.8, 121.2)
- moved TP1 12.1 mm to (120.5, 126.0)
- moved F1 8.49 mm to (116.0, 90.8)
- moved F2 7.72 mm to (127.0, 90.8)
- moved LOGO2 2.64 mm to (172.5, 75.2)
- moved G*** 2.46 mm to (183.2, 121.2)
- moved G*** 2.24 mm to (182.0, 77.0)
- moved TP5 1.70 mm to (160.2, 79.5)
- moved J1 1.07 mm to (120.0, 84.0)
Routing:
- net ISO_5V: track 16.8 -> 15.1 mm
- net LVGND: vias 99 -> 88
- net HVGND: vias 107 -> 92
Other:
- board text added: "Active Precharge Rev B Gavin Wang March 2026"
- board text added: "HV GND"
- board text added: "High Voltage!!!!"
- board text added: "Low Voltage!"
- board text added: "Nah I'd Short"
- board text removed: "Active Precharge Rev B Gavin Wang December 2025"
- board text removed: "HV"
- board text removed: "LV"
